Commit message: Adding .stl file, and correcting typo in name

File: catkin_ws/src/trog_description/urdf/decorations.urdf.xacro (robot description, xacro)
@@ -34,5 +34,5 @@
             <origin xyz="0 0 0" rpy="0 0 0" />
             <geometry>
-              <mesh filename="package://husky_description/meshes/top_plate_2.dae" />
+              <mesh filename="package://trog_description/meshes/top_plate.dae" />
             </geometry>
           </visual>
@@ -40,5 +40,5 @@
             <origin xyz="0 0 0" rpy="0 0 0"/>
             <geometry>
-              <mesh filename="package://husky_description/meshes/top_plate.stl" />
+              <mesh filename="package://trog_description/meshes/top_plate.stl" />
             </geometry>
           </collision>
